File: Hardware/PCB/spro2/nps.kicad_sch (KiCad schematic)
At the start: 3 parts

Commit message: Temp circ fixed, added footprint for MAX6
Parts:
- U4: footprint (none) -> Package_DIP:DIP-8_W7.62mm
Changed lines of the file:
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@@
 			)
 		)
-		(property "Footprint" ""
+		(property "Footprint" "Package_DIP:DIP-8_W7.62mm"
 			(at 146.05 92.71 0)
 			(effects

Commit message: finish schematic
Connections:
- net +5V renamed NPS_IN
- net -5V renamed NPS_OUT
Changed lines of the file:
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@@
-	(wire
-		(pts
-			(xy 171.45 100.33) (xy 171.45 88.9)
-		)
-		(stroke
-			(width 0)
-			(type default)
-		)
-	)
 	(wire
 		(pts
@@
 		)
 	)
-	(symbol
-		(lib_id "power:-5V")
-		(at 171.45 88.9 0)
-		(unit 1)
-		(exclude_from_sim no)
-		(in_bom yes)
-		(on_board yes)
-		(dnp no)
-		(property "Reference" "#PWR05"
-			(at 171.45 92.71 0)
-			(effects
-				(font
-					(size 1.27 1.27)
-				)
-				(hide yes)
+	(hierarchical_label "NPS_IN"
+		(shape input)
+		(at 165.1 88.9 0)
+		(fields_autoplaced yes)
+		(effects
+			(font
+				(size 1.27 1.27)
 			)
-		)
-		(property "Value" "-5V"
-			(at 171.704 84.836 0)
-			(effects
-				(font
-					(size 1.27 1.27)
-				)
-			)
-		)
-		(property "Footprint" ""
-			(at 171.45 88.9 0)
-			(effects
-				(font
-					(size 1.27 1.27)
-				)
-				(hide yes)
-			)
-		)
-		(property "Datasheet" ""
-			(at 171.45 88.9 0)
-			(effects
-				(font
-					(size 1.27 1.27)
-				)
-				(hide yes)
-			)
-		)
-		(property "Description" "Power symbol creates a global label with name \"-5V\""
-			(at 171.45 88.9 0)
-			(effects
-				(font
-					(size 1.27 1.27)
-				)
-				(hide yes)
-			)
-		)
-		(pin "1"
-		)
-		(instances
-			(project "spro2"
-				(path "/edfea366-2226-45cc-893f-1155e0ffe333/64df08b9-4000-4721-b83a-705bd7162f6e/93c1714d-5bc5-4522-b05d-5ce4f6256433"
-					(reference "#PWR05")
-					(unit 1)
-				)
-			)
+			(justify left)
 		)
 	)
-	(symbol
-		(lib_id "power:+5V")
-		(at 165.1 88.9 0)
-		(unit 1)
-		(exclude_from_sim no)
-		(in_bom yes)
-		(on_board yes)
-		(dnp no)
+	(hierarchical_label "NPS_OUT"
+		(shape output)
+		(at 171.45 100.33 0)
 		(fields_autoplaced yes)
-		(property "Reference" "#PWR04"
-			(at 165.1 92.71 0)
-			(effects
-				(font
-					(size 1.27 1.27)
-				)
-				(hide yes)
+		(effects
+			(font
+				(size 1.27 1.27)
 			)
-		)
-		(property "Value" "+5V"
-			(at 165.1 83.82 0)
-			(effects
-				(font
-					(size 1.27 1.27)
-				)
-			)
-		)
-		(property "Footprint" ""
-			(at 165.1 88.9 0)
-			(effects
-				(font
-					(size 1.27 1.27)
-				)
-				(hide yes)
-			)
-		)
-		(property "Datasheet" ""
-			(at 165.1 88.9 0)
-			(effects
-				(font
-					(size 1.27 1.27)
-				)
-				(hide yes)
-			)
-		)
-		(property "Description" "Power symbol creates a global label with name \"+5V\""
-			(at 165.1 88.9 0)
-			(effects
-				(font
-					(size 1.27 1.27)
-				)
-				(hide yes)
-			)
-		)
-		(pin "1"
-		)
-		(instances
-			(project ""
-				(path "/edfea366-2226-45cc-893f-1155e0ffe333/64df08b9-4000-4721-b83a-705bd7162f6e/93c1714d-5bc5-4522-b05d-5ce4f6256433"
-					(reference "#PWR04")
-					(unit 1)
-				)
-			)
+			(justify left)
 		)
 	)

Commit message: Hopefully last version of PCB
Parts:
- C12, C13: footprint (none) -> CP_Radial_D10.0mm_P5.00mm
Changed lines of the file:
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@@
+		)
+	)
+	(label "-5V"
+		(at 165.1 100.33 0)
+		(fields_autoplaced yes)
+		(effects
+			(font
+				(size 1.27 1.27)
+			)
+			(justify left bottom)
 		)
 	)
@@
 		(on_board yes)
 		(dnp no)
-		(fields_autoplaced yes)
 		(property "Reference" "#PWR03"
 			(at 134.62 105.41 0)
@@
 		)
 		(property "Value" "GND"
-			(at 134.62 104.14 0)
+			(at 137.922 101.092 0)
 			(effects
 				(font
@@
 			)
 		)
-		(property "Footprint" ""
+		(property "Footprint" "CP_Radial_D10.0mm_P5.00mm"
 			(at 166.0652 114.3 0)
 			(effects
@@
 			)
 		)
-		(property "Footprint" ""
+		(property "Footprint" "CP_Radial_D10.0mm_P5.00mm"
 			(at 125.4252 102.87 0)
 			(effects
