File: Hardware/PCB/spro2/hum_sensor.kicad_sch (KiCad schematic)
At the start: 20 parts, among them J3 Humidity sensor, U3 TL074

Commit message: finish schematic
Changed lines of the file:
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@@
-	(wire
-		(pts
-			(xy 73.66 158.75) (xy 73.66 160.02)
-		)
-		(stroke
-			(width 0)
-			(type default)
-		)
-	)
 	(wire
 		(pts
@@
 	(wire
 		(pts
+			(xy 85.09 158.75) (xy 85.09 157.48)
+		)
+		(stroke
+			(width 0)
+			(type default)
+		)
+	)
+	(wire
+		(pts
 			(xy 142.24 78.74) (xy 146.05 78.74)
 		)
@@
 	(wire
 		(pts
+			(xy 73.66 158.75) (xy 85.09 158.75)
+		)
+		(stroke
+			(width 0)
+			(type default)
+		)
+	)
+	(wire
+		(pts
 			(xy 119.38 78.74) (xy 129.54 78.74)
 		)
@@
 	(wire
 		(pts
+			(xy 228.6 139.7) (xy 228.6 140.97)
+		)
+		(stroke
+			(width 0)
+			(type default)
+		)
+	)
+	(wire
+		(pts
 			(xy 215.9 74.93) (xy 208.28 74.93)
 		)
@@
 	(wire
 		(pts
+			(xy 257.81 139.7) (xy 257.81 140.97)
+		)
+		(stroke
+			(width 0)
+			(type default)
+		)
+	)
+	(wire
+		(pts
 			(xy 102.87 101.6) (xy 101.6 101.6)
 		)
@@
 	(wire
 		(pts
+			(xy 252.73 140.97) (xy 257.81 140.97)
+		)
+		(stroke
+			(width 0)
+			(type default)
+		)
+	)
+	(wire
+		(pts
 			(xy 83.82 114.3) (xy 83.82 115.57)
 		)
@@
 		(pts
 			(xy 101.6 109.22) (xy 102.87 109.22)
+		)
+		(stroke
+			(width 0)
+			(type default)
+		)
+	)
+	(wire
+		(pts
+			(xy 228.6 140.97) (xy 233.68 140.97)
 		)
 		(stroke
@@
 		)
 	)
-	(symbol
-		(lib_id "power:-5V")
-		(at 73.66 160.02 180)
-		(unit 1)
-		(exclude_from_sim no)
-		(in_bom yes)
-		(on_board yes)
-		(dnp no)
-		(property "Reference" "#PWR020"
-			(at 73.66 156.21 0)
-			(effects
-				(font
-					(size 1.27 1.27)
-				)
-				(hide yes)
-			)
-		)
-		(property "Value" "-5V"
-			(at 73.406 164.084 0)
-			(effects
-				(font
-					(size 1.27 1.27)
-				)
-			)
-		)
-		(property "Footprint" ""
-			(at 73.66 160.02 0)
-			(effects
-				(font
-					(size 1.27 1.27)
-				)
-				(hide yes)
-			)
-		)
-		(property "Datasheet" ""
-			(at 73.66 160.02 0)
-			(effects
-				(font
-					(size 1.27 1.27)
-				)
-				(hide yes)
-			)
-		)
-		(property "Description" "Power symbol creates a global label with name \"-5V\""
-			(at 73.66 160.02 0)
-			(effects
-				(font
-					(size 1.27 1.27)
-				)
-				(hide yes)
-			)
-		)
-		(pin "1"
-		)
-		(instances
-			(project "spro2"
-				(path "/edfea366-2226-45cc-893f-1155e0ffe333/64df08b9-4000-4721-b83a-705bd7162f6e"
-					(reference "#PWR020")
-					(unit 1)
-				)
-			)
+	(hierarchical_label "NPS_OUT"
+		(shape output)
+		(at 252.73 140.97 180)
+		(fields_autoplaced yes)
+		(effects
+			(font
+				(size 1.27 1.27)
+			)
+			(justify right)
+		)
+	)
+	(hierarchical_label "NPS_IN"
+		(shape output)
+		(at 233.68 140.97 0)
+		(fields_autoplaced yes)
+		(effects
+			(font
+				(size 1.27 1.27)
+			)
+			(justify left)
 		)
 	)
@@
 	(symbol
 		(lib_id "power:+5V")
+		(at 228.6 139.7 0)
+		(unit 1)
+		(exclude_from_sim no)
+		(in_bom yes)
+		(on_board yes)
+		(dnp no)
+		(property "Reference" "#PWR04"
+			(at 228.6 143.51 0)
+			(effects
+				(font
+					(size 1.27 1.27)
+				)
+				(hide yes)
+			)
+		)
+		(property "Value" "+5V"
+			(at 228.6 135.89 0)
+			(effects
+				(font
+					(size 1.27 1.27)
+				)
+			)
+		)
+		(property "Footprint" ""
+			(at 228.6 139.7 0)
+			(effects
+				(font
+					(size 1.27 1.27)
+				)
+				(hide yes)
+			)
+		)
+		(property "Datasheet" ""
+			(at 228.6 139.7 0)
+			(effects
+				(font
+					(size 1.27 1.27)
+				)
+				(hide yes)
+			)
+		)
+		(property "Description" "Power symbol creates a global label with name \"+5V\""
+			(at 228.6 139.7 0)
+			(effects
+				(font
+					(size 1.27 1.27)
+				)
+				(hide yes)
+			)
+		)
+		(pin "1"
+		)
+		(instances
+			(project "spro2"
+				(path "/edfea366-2226-45cc-893f-1155e0ffe333/64df08b9-4000-4721-b83a-705bd7162f6e"
+					(reference "#PWR04")
+					(unit 1)
+				)
+			)
+		)
+	)
+	(symbol
+		(lib_id "power:+5V")
 		(at 73.66 142.24 0)
 		(unit 1)
@@
 	)
 	(symbol
+		(lib_id "power:+5V")
+		(at 257.81 139.7 0)
+		(unit 1)
+		(exclude_from_sim no)
+		(in_bom yes)
+		(on_board yes)
+		(dnp no)
+		(property "Reference" "#PWR020"
+			(at 257.81 143.51 0)
+			(effects
+				(font
+					(size 1.27 1.27)
+				)
+				(hide yes)
+			)
+		)
+		(property "Value" "-5V"
+			(at 257.81 135.89 0)
+			(effects
+				(font
+					(size 1.27 1.27)
+				)
+			)
+		)
+		(property "Footprint" ""
+			(at 257.81 139.7 0)
+			(effects
+				(font
+					(size 1.27 1.27)
+				)
+				(hide yes)
+			)
+		)
+		(property "Datasheet" ""
+			(at 257.81 139.7 0)
+			(effects
+				(font
+					(size 1.27 1.27)
+				)
+				(hide yes)
+			)
+		)
+		(property "Description" "Power symbol creates a global label with name \"+5V\""
+			(at 257.81 139.7 0)
+			(effects
+				(font
+					(size 1.27 1.27)
+				)
+				(hide yes)
+			)
+		)
+		(pin "1"
+		)
+		(instances
+			(project "spro2"
+				(path "/edfea366-2226-45cc-893f-1155e0ffe333/64df08b9-4000-4721-b83a-705bd7162f6e"
+					(reference "#PWR020")
+					(unit 1)
+				)
+			)
+		)
+	)
+	(symbol
 		(lib_id "Amplifier_Operational:TL074")
 		(at 76.2 151.13 0)
@@
 	)
 	(symbol
+		(lib_id "power:+5V")
+		(at 85.09 157.48 0)
+		(unit 1)
+		(exclude_from_sim no)
+		(in_bom yes)
+		(on_board yes)
+		(dnp no)
+		(property "Reference" "#PWR05"
+			(at 85.09 161.29 0)
+			(effects
+				(font
+					(size 1.27 1.27)
+				)
+				(hide yes)
+			)
+		)
+		(property "Value" "-5V"
+			(at 85.09 153.67 0)
+			(effects
+				(font
+					(size 1.27 1.27)
+				)
+			)
+		)
+		(property "Footprint" ""
+			(at 85.09 157.48 0)
+			(effects
+				(font
+					(size 1.27 1.27)
+				)
+				(hide yes)
+			)
+		)
+		(property "Datasheet" ""
+			(at 85.09 157.48 0)
+			(effects
+				(font
+					(size 1.27 1.27)
+				)
+				(hide yes)
+			)
+		)
+		(property "Description" "Power symbol creates a global label with name \"+5V\""
+			(at 85.09 157.48 0)
+			(effects
+				(font
+					(size 1.27 1.27)
+				)
+				(hide yes)
+			)
+		)
+		(pin "1"
+		)
+		(instances
+			(project "spro2"
+				(path "/edfea366-2226-45cc-893f-1155e0ffe333/64df08b9-4000-4721-b83a-705bd7162f6e"
+					(reference "#PWR05")
+					(unit 1)
+				)
+			)
+		)
+	)
+	(symbol
 		(lib_id "Device:C")
 		(at 77.47 110.49 0)
@@
 	(sheet
 		(at 233.68 137.795)
-		(size 12.7 3.81)
+		(size 19.05 6.985)
 		(fields_autoplaced yes)
 		(stroke
@@
 		)
 		(property "Sheetfile" "nps.kicad_sch"
-			(at 233.68 142.1896 0)
-			(effects
-				(font
+			(at 233.68 145.3646 0)
+			(effects
+				(font

Commit message: Hopefully last version of PCB
Parts:
- added C8, C9: 100u, Capacitor_THT:CP_Radial_D10.0mm_P5.00mm, symbol Device:C_Polarized
- added U4: ~, Package_DIP:DIP-8_W7.62mm, symbol nps:MAX660CPA+
- C10: renamed from C4; footprint C_Rect_L7.2mm_W8.5mm_P5.00mm_FKP2_FKP2_MKS2_MKP2 -> Capacitor_THT:C_Rect_L13.0mm_W5.0mm_P10.00mm_FKS3_FKP3_MKS4
- C11: renamed from C10; footprint C_Rect_L7.2mm_W3.0mm_P5.00mm_FKS2_FKP2_MKS2_MKP2 -> Capacitor_THT:C_Rect_L7.2mm_W2.5mm_P5.00mm_FKS2_FKP2_MKS2_MKP2
- C12: renamed from C5; footprint C_Rect_L7.2mm_W8.5mm_P5.00mm_FKP2_FKP2_MKS2_MKP2 -> Capacitor_THT:C_Rect_L13.0mm_W5.0mm_P10.00mm_FKS3_FKP3_MKS4
- C13: renamed from C11; footprint C_Rect_L7.2mm_W3.0mm_P5.00mm_FKS2_FKP2_MKS2_MKP2 -> Capacitor_THT:C_Rect_L7.2mm_W2.5mm_P5.00mm_FKS2_FKP2_MKS2_MKP2
- renumbered J3 to J2, R9 to R11, R10 to R12, R11 to R13, R12 to R14, R13 to R15, R14 to R16, R15 to R17, R16 to R18, R17 to R19, R18 to R20
Connections:
- net +5V: now also U4.8 (V+)
- net -5V: now also C9.1, U4.5 (OUT)
- net GND: now also C9.2, U4.3 (GND)
- new net: C8.1, U4.2 (CAP+)
- new net: C8.2, U4.4 (CAP-)
- no-connect marks 0 -> 3
Other:
- removed sheet Negative power supply
- note added: "220n: C_Rect_L7.2mm_W3.5mm_P5.00mm_FKS2_FKP2_MKS2_MKP2"
- moved on the sheet: U3E

Commit message: pcb finalized
Connections:
- net -5V: now also C9.2; no longer C9.1
- net GND: now also C9.1; no longer C9.2
Other:
- moved on the sheet: C9

Commit message: Finished PCB
Parts:
- J2: footprint Diplomna:connector_2p -> SPRO_lib:connector_2p
Changed lines of the file:
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@@
 			)
 		)
-		(property "Footprint" "Diplomna:connector_2p"
+		(property "Footprint" "SPRO_lib:connector_2p"
 			(at 129.54 73.66 0)
 			(effects

Commit message: Final scheamtic mega trust
Connections:
- net GND: now also U3.10 (+), U3.5 (+); no longer U3.6 (-), U3.9 (-)
- net at D1.2 (A), D2.1 (K), R11.2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: now also U3.2 (-); no longer U3.3 (+)
- net at C10.1, C11.1, C12.2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: now also U3.3 (+); no longer U3.2 (-)
- net at R17.2, R19.2, R20.1: now also U3.9 (-); no longer U3.10 (+)
- net at D3.1 (K), R16.2, R18.1: now also U3.6 (-); no longer U3.5 (+)
Changed lines of the file:
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@@
 		(lib_id "Amplifier_Operational:TL074")
 		(at 223.52 77.47 0)
+		(mirror x)
 		(unit 3)
 		(exclude_from_sim no)
@@
 		(fields_autoplaced yes)
 		(property "Reference" "U3"
-			(at 223.52 67.31 0)
+			(at 223.52 87.63 0)
 			(effects
 				(font
@@
 		)
 		(property "Value" "TL074"
-			(at 223.52 69.85 0)
+			(at 223.52 85.09 0)
 			(effects
 				(font
@@
 		)
 		(property "Footprint" "SPRO_lib:DIP794W53P254L1930H508Q14N"
-			(at 222.25 74.93 0)
+			(at 222.25 80.01 0)
 			(effects
 				(font
@@
 		)
 		(property "Datasheet" "http://www.ti.com/lit/ds/symlink/tl071.pdf"
-			(at 224.79 72.39 0)
+			(at 224.79 82.55 0)
 			(effects
 				(font
@@
 		(lib_id "Amplifier_Operational:TL074")
 		(at 180.34 109.22 0)
+		(mirror x)
 		(unit 2)
 		(exclude_from_sim no)
@@
 		(fields_autoplaced yes)
 		(property "Reference" "U3"
-			(at 180.34 99.06 0)
+			(at 180.34 119.38 0)
 			(effects
 				(font
@@
 		)
 		(property "Value" "TL074"
-			(at 180.34 101.6 0)
+			(at 180.34 116.84 0)
 			(effects
 				(font
@@
 		)
 		(property "Footprint" "SPRO_lib:DIP794W53P254L1930H508Q14N"
-			(at 179.07 106.68 0)
+			(at 179.07 111.76 0)
 			(effects
 				(font
@@
 		)
 		(property "Datasheet" "http://www.ti.com/lit/ds/symlink/tl071.pdf"
-			(at 181.61 104.14 0)
+			(at 181.61 114.3 0)
 			(effects
 				(font
@@
 		(lib_id "Amplifier_Operational:TL074")
 		(at 91.44 78.74 0)
+		(mirror x)
 		(unit 1)
 		(exclude_from_sim no)
@@
 		(fields_autoplaced yes)
 		(property "Reference" "U3"
-			(at 91.44 68.58 0)
+			(at 91.44 88.9 0)
 			(effects
 				(font
@@
 		)
 		(property "Value" "TL074"
-			(at 91.44 71.12 0)
+			(at 91.44 86.36 0)
 			(effects
 				(font
@@
 		)
 		(property "Footprint" "SPRO_lib:DIP794W53P254L1930H508Q14N"
-			(at 90.17 76.2 0)
+			(at 90.17 81.28 0)
 			(effects
 				(font
@@
 		)
 		(property "Datasheet" "http://www.ti.com/lit/ds/symlink/tl071.pdf"
-			(at 92.71 73.66 0)
-			(effects
-				(font
+			(at 92.71 83.82 0)
+			(effects
+				(font
